Commit message: fixed gazebo path and render in Gazebo and Rviz, portable version

File: urdf/camera.xacro (robot description, xacro)
@@ -15,5 +15,6 @@
             <geometry>
                 <!-- <box size="0.01 0.03 0.03" /> -->
-                <mesh filename="package://ur_yt_sim/meshes/sensors/camera/kinetic.stl"/>
+                <!-- <mesh filename="package://ur_yt_sim/meshes/sensors/camera/kinetic.stl"/> -->
+                <mesh filename="file://${URYT}/meshes/sensors/camera/kinetic.stl"/>
             </geometry>
             <material name="red"/>
@@ -21,5 +22,6 @@
         <collision>
             <geometry>
-                <mesh filename="package://ur_yt_sim/meshes/sensors/camera/kinetic.dae"/>
+                <!-- <mesh filename="package://ur_yt_sim/meshes/sensors/camera/kinetic.dae"/> -->
+                <mesh filename="file://${URYT}/meshes/sensors/camera/kinetic.dae"/>
             </geometry>
         </collision>
@@ -38,41 +40,17 @@
     </joint>
     <gazebo reference="camera_link">
-        <visual>
-            <geometry>
-                <mesh>
-                    <uri>package://ur_yt_sim/meshes/sensors/camera/kinetic.stl</uri>
-                </mesh>
-            </geometry>
-            <material>Gazebo/Red</material>
-        </visual>
-        <!-- <material>Gazebo/Red</material> -->
         <sensor name="camera" type="depth">
-            <pose> 0 0 0 0 0 0 </pose>
+            <pose>0 0 0 0 0 0</pose>
             <visualize>true</visualize>
             <update_rate>10</update_rate>
             <camera>
-                <horizontal_fov>1.089</horizontal_fov>
-                <image>
-                    <format>R8G8B8</format>
-                    <width>640</width>
-                    <height>480</height>
-                </image>
-                <clip>
-                    <near>0.05</near>
-                    <far>8</far>
-                </clip>
+            <horizontal_fov>1.089</horizontal_fov>
+            <image><format>R8G8B8</format><width>640</width><height>480</height></image>
+            <clip><near>0.05</near><far>8</far></clip>
             </camera>
-            <plugin name="camera_controller" filename="libgazebo_ros_camera.so" >
-                <frame_name>camera_optical_link</frame_name>
+            <plugin name="camera_controller" filename="libgazebo_ros_camera.so">
+            <frame_name>camera_optical_link</frame_name>
             </plugin>
         </sensor>
     </gazebo>
-    <gazebo reference="camera_link">
-        <visual>
-            <geometry>
-                <mesh filename="package://ur_yt_sim/meshes/sensors/camera/kinetic.stl"/>
-            </geometry>
-            <material>Gazebo/Red</material>
-        </visual>
-    </gazebo>
 </robot>

File: urdf/robotiq_gripper_macro.xacro (robot description, xacro)
@@ -43,10 +43,12 @@
             <visual>
                 <geometry>
-                    <mesh filename="package://robotiq_description/meshes/visual/2f_85/robotiq_base.dae" />
-                </geometry>
-            </visual>
-            <collision>
-                <geometry>
-                    <mesh filename="package://robotiq_description/meshes/collision/2f_85/robotiq_base.stl" />
+                    <!-- <mesh filename="package://robotiq_description/meshes/visual/2f_85/robotiq_base.dae" /> -->
+                    <mesh filename="file://${ROBI}/meshes/visual/2f_85/robotiq_base.dae"/>
+                </geometry>
+            </visual>
+            <collision>
+                <geometry>
+                    <!-- <mesh filename="package://robotiq_description/meshes/collision/2f_85/robotiq_base.stl" /> -->
+                    <mesh filename="file://${ROBI}/meshes/collision/2f_85/robotiq_base.stl" />
                 </geometry>
             </collision>
@@ -60,10 +62,12 @@
             <visual>
                 <geometry>
-                    <mesh filename="package://robotiq_description/meshes/visual/2f_85/left_knuckle.dae" />
-                </geometry>
-            </visual>
-            <collision>
-                <geometry>
-                    <mesh filename="package://robotiq_description/meshes/collision/2f_85/left_knuckle.stl" />
+                    <!-- <mesh filename="package://robotiq_description/meshes/visual/2f_85/left_knuckle.dae" /> -->
+                    <mesh filename="file://${ROBI}/meshes/visual/2f_85/left_knuckle.dae" />
+                </geometry>
+            </visual>
+            <collision>
+                <geometry>
+                    <!-- <mesh filename="package://robotiq_description/meshes/collision/2f_85/left_knuckle.stl" /> -->
+                    <mesh filename="file://${ROBI}/meshes/collision/2f_85/left_knuckle.stl" />
                 </geometry>
             </collision>
@@ -77,10 +81,12 @@
             <visual>
                 <geometry>
-                    <mesh filename="package://robotiq_description/meshes/visual/2f_85/right_knuckle.dae" />
-                </geometry>
-            </visual>
-            <collision>
-                <geometry>
-                    <mesh filename="package://robotiq_description/meshes/collision/2f_85/right_knuckle.stl" />
+                    <!-- <mesh filename="package://robotiq_description/meshes/visual/2f_85/right_knuckle.dae" /> -->
+                    <mesh filename="file://${ROBI}/meshes/visual/2f_85/right_knuckle.dae" />
+                </geometry>
+            </visual>
+            <collision>
+                <geometry>
+                    <!-- <mesh filename="package://robotiq_description/meshes/collision/2f_85/right_knuckle.stl" /> -->
+                    <mesh filename="file://${ROBI}/meshes/collision/2f_85/right_knuckle.stl" />
                 </geometry>
             </collision>
@@ -94,10 +100,12 @@
             <visual>
                 <geometry>
-                    <mesh filename="package://robotiq_description/meshes/visual/2f_85/left_finger.dae" />
-                </geometry>
-            </visual>
-            <collision>
-                <geometry>
-                    <mesh filename="package://robotiq_description/meshes/collision/2f_85/left_finger.stl" />
+                    <!-- <mesh filename="package://robotiq_description/meshes/visual/2f_85/left_finger.dae" /> -->
+                    <mesh filename="file://${ROBI}/meshes/visual/2f_85/left_finger.dae" />
+                </geometry>
+            </visual>
+            <collision>
+                <geometry>
+                    <!-- <mesh filename="package://robotiq_description/meshes/collision/2f_85/left_finger.stl" /> -->
+                    <mesh filename="file://${ROBI}/meshes/collision/2f_85/left_finger.stl" />
                 </geometry>
             </collision>
@@ -111,10 +119,12 @@
             <visual>
                 <geometry>
-                    <mesh filename="package://robotiq_description/meshes/visual/2f_85/right_finger.dae" />
-                </geometry>
-            </visual>
-            <collision>
-                <geometry>
-                    <mesh filename="package://robotiq_description/meshes/collision/2f_85/right_finger.stl" />
+                    <!-- <mesh filename="package://robotiq_description/meshes/visual/2f_85/right_finger.dae" /> -->
+                    <mesh filename="file://${ROBI}/meshes/visual/2f_85/right_finger.dae" />
+                </geometry>
+            </visual>
+            <collision>
+                <geometry>
+                    <!-- <mesh filename="package://robotiq_description/meshes/collision/2f_85/right_finger.stl" /> -->
+                    <mesh filename="file://${ROBI}/meshes/collision/2f_85/right_finger.stl" />
                 </geometry>
             </collision>
@@ -128,10 +138,12 @@
             <visual>
                 <geometry>
-                    <mesh filename="package://robotiq_description/meshes/visual/2f_85/left_inner_knuckle.dae" />
-                </geometry>
-            </visual>
-            <collision>
-                <geometry>
-                    <mesh filename="package://robotiq_description/meshes/collision/2f_85/left_inner_knuckle.stl" />
+                    <!-- <mesh filename="package://robotiq_description/meshes/visual/2f_85/left_inner_knuckle.dae" /> -->
+                    <mesh filename="file://${ROBI}/meshes/visual/2f_85/left_inner_knuckle.dae" />
+                </geometry>
+            </visual>
+            <collision>
+                <geometry>
+                    <!-- <mesh filename="package://robotiq_description/meshes/collision/2f_85/left_inner_knuckle.stl" /> -->
+                    <mesh filename="file://${ROBI}/meshes/collision/2f_85/left_inner_knuckle.stl" />
                 </geometry>
             </collision>
@@ -145,10 +157,12 @@
             <visual>
                 <geometry>
-                    <mesh filename="package://robotiq_description/meshes/visual/2f_85/right_inner_knuckle.dae" />
-                </geometry>
-            </visual>
-            <collision>
-                <geometry>
-                    <mesh filename="package://robotiq_description/meshes/collision/2f_85/right_inner_knuckle.stl" />
+                    <!-- <mesh filename="package://robotiq_description/meshes/visual/2f_85/right_inner_knuckle.dae" /> -->
+                    <mesh filename="file://${ROBI}/meshes/visual/2f_85/right_inner_knuckle.dae" />
+                </geometry>
+            </visual>
+            <collision>
+                <geometry>
+                    <!-- <mesh filename="package://robotiq_description/meshes/collision/2f_85/right_inner_knuckle.stl" /> -->
+                    <mesh filename="file://${ROBI}/meshes/collision/2f_85/right_inner_knuckle.stl" />
                 </geometry>
             </collision>
@@ -162,10 +176,12 @@
             <visual>
                 <geometry>
-                    <mesh filename="package://robotiq_description/meshes/visual/2f_85/left_finger_tip.dae" />
-                </geometry>
-            </visual>
-            <collision>
-                <geometry>
-                    <mesh filename="package://robotiq_description/meshes/collision/2f_85/left_finger_tip.stl" />
+                    <!-- <mesh filename="package://robotiq_description/meshes/visual/2f_85/left_finger_tip.dae" /> -->
+                    <mesh filename="file://${ROBI}/meshes/visual/2f_85/left_finger_tip.dae" />
+                </geometry>
+            </visual>
+            <collision>
+                <geometry>
+                    <!-- <mesh filename="package://robotiq_description/meshes/collision/2f_85/left_finger_tip.stl" /> -->
+                    <mesh filename="file://${ROBI}/meshes/collision/2f_85/left_finger_tip.stl" />
                 </geometry>
                 <surface>
@@ -197,10 +213,12 @@
             <visual>
                 <geometry>
-                    <mesh filename="package://robotiq_description/meshes/visual/2f_85/right_finger_tip.dae" />
-                </geometry>
-            </visual>
-            <collision>
-                <geometry>
-                    <mesh filename="package://robotiq_description/meshes/collision/2f_85/right_finger_tip.stl" />
+                    <!-- <mesh filename="package://robotiq_description/meshes/visual/2f_85/right_finger_tip.dae" /> -->
+                    <mesh filename="file://${ROBI}/meshes/visual/2f_85/right_finger_tip.dae" />
+                </geometry>
+            </visual>
+            <collision>
+                <geometry>
+                    <!-- <mesh filename="package://robotiq_description/meshes/collision/2f_85/right_finger_tip.stl" /> -->
+                    <mesh filename="file://${ROBI}/meshes/collision/2f_85/right_finger_tip.stl" />
                 </geometry>
                 <surface>

File: urdf/ur5_camera_gripper.urdf.xacro (robot description, xacro)
@@ -4,4 +4,8 @@
    <xacro:arg name="name" default="ur"/>
    <!-- import main macro -->
+   <xacro:property name="URYT" value="$(find ur_yt_sim)"/>
+   <xacro:property name="ROBI" value="$(find robotiq_description)"/>
+   <!-- <xacro:include filename="$(find-pkg-share ur_yt_sim)/urdf/camera.xacro"/>
+   <xacro:include filename="$(find-pkg-share ur_yt_sim)/urdf/ur5_macro.xacro"/> -->
    <xacro:include filename="$(find ur_yt_sim)/urdf/camera.xacro"/>
    <xacro:include filename="$(find ur_yt_sim)/urdf/ur5_macro.xacro"/>
@@ -46,6 +50,8 @@
    <xacro:arg name="sim_ignition" default="false" />
    <xacro:arg name="simulation_controllers" default="$(find ur_yt_sim)/config/ur5_controllers_gripper.yaml" />
+   <!-- <xacro:arg name="simulation_controllers" default="$(find-pkg-share ur_yt_sim)/config/ur5_controllers_gripper.yaml" /> -->
    <!-- initial position for simulations (Fake Hardware, Gazebo, Ignition) -->
    <xacro:arg name="initial_positions_file" default="$(find ur_yt_sim)/config/initial_positions.yaml"/>
+   <!-- <xacro:arg name="initial_positions_file" default="$(find-pkg-share ur_yt_sim)/config/initial_positions.yaml"/> -->
    <!-- convert to property to use substitution in function -->
    <xacro:property name="initial_positions_file" default="$(arg initial_positions_file)"/>
@@ -139,10 +145,15 @@
     </gazebo>
   </xacro:if>
-  <xacro:arg name="use_fake_hardware" default="true" />
+  <xacro:arg name="use_fake_hardware" default="false" />
   <xacro:arg name="com_port" default="/dev/ttyUSB0" />
   <!-- Import macros -->
   <xacro:include filename="$(find ur_yt_sim)/urdf/robotiq_gripper_macro.xacro" />
-  <xacro:robotiq_gripper name="RobotiqGripperHardwareInterface" prefix="" parent="tool0" use_fake_hardware="$(arg use_fake_hardware)" com_port="$(arg com_port)" sim_gazebo="$(arg sim_gazebo)">
-    <origin xyz="0 0 0" rpy="0 0 0" />
+  <xacro:robotiq_gripper
+    name="RobotiqGripperHardwareInterface"
+    prefix=""
+    parent="tool0"
+    sim_gazebo="$(arg sim_gazebo)"
+    com_port="$(arg com_port)">
+    <origin xyz="0 0 0" rpy="0 0 0"/>
   </xacro:robotiq_gripper>
 </robot>
